File: template/template.kicad_pcb (KiCad board)
At the start: 2 copper layers, 2 parts

Commit message: Template ready
Parts:
- added R1: 90, Resistor_THT:R_Axial_DIN0309_L9.0mm_D3.2mm_P15.24mm_Horizontal, F.Cu at (144.5, 84.7)
- added S1: TS02-66-70-BK-160-LCR-D, Robot Uprising:SW_TS02-66-70-BK-160-LCR-D, F.Cu at (147.8, 91.8)
- BT1: footprint -Robot Uprising:BAT-HLD-005-THM -> Robot Uprising:BAT-HLD-005-THM

Commit message: Cleanup
Parts:
- added D2: LED, LED_THT:LED_D5.0mm, F.Cu at (140.2, 79.7)
- added R2: 47, Resistor_THT:R_Axial_DIN0309_L9.0mm_D3.2mm_P15.24mm_Horizontal, F.Cu at (114.1, 96.8)
- BT1: value BAT-HLD-005-THM -> BT_BAT-HLD-005-THM; footprint Robot Uprising:BAT-HLD-005-THM -> Robot Uprising:BT_BAT-HLD-005-THM
- R1: value 90 -> 47
- S1: value TS02-66-70-BK-160-LCR-D -> S_TS02-66-70-BK-160-LCR-D; footprint Robot Uprising:SW_TS02-66-70-BK-160-LCR-D -> Robot Uprising:S_TS02-66-70-BK-160-LCR-D
- moved D1 36.9 mm to (140.2, 72.2)
- moved R1 31.4 mm to (114.1, 92.0)
- moved S1 12.4 mm to (135.7, 94.3)
- moved BT1 8.77 mm to (125.1, 79.5)

Commit message: pre-event-3
Workshop files ready
Parts:
- removed BT1: BT_BAT-HLD-005-THM, Robot Uprising:BT_BAT-HLD-005-THM
- removed D1, D2: LED, LED_THT:LED_D5.0mm
- removed R1, R2: 47, Resistor_THT:R_Axial_DIN0309_L9.0mm_D3.2mm_P15.24mm_Horizontal
- removed S1: S_TS02-66-70-BK-160-LCR-D, Robot Uprising:S_TS02-66-70-BK-160-LCR-D
